File: kicad/transmitter/transmitter.kicad_sch (KiCad schematic)
At the start: 16 parts, among them J1 Barrel_Jack_MountingPin, Q1 IRF740, SW1 SW_SPST

Commit message: Schematic update
Parts:
- C1: value C -> 100n
- C2: value C_Polarized -> 100u
- Q1: value IRF740 -> IRF540
- R1: value 1K8 -> 1K
Other:
- note added: "Two Dogs Motorsport"
Changed lines of the file:
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@@
     (stroke (width 0) (type default))
+  )
+  (text "Two Dogs Motorsport" (at 201.93 176.53 0)
+    (effects (font (size 4 4) (thickness 0.8) bold (color 132 0 0 1)) (justify left bottom))
   )
   (symbol (lib_id "Device:LED") (at 194.31 60.96 90) (unit 1)
@@
       (effects (font (size 1.27 1.27)) (justify left))
     )
-    (property "Value" "IRF740" (at 198.12 81.28 0)
+    (property "Value" "IRF540" (at 198.12 81.28 0)
       (effects (font (size 1.27 1.27)) (justify left))
     )
@@
       (effects (font (size 1.27 1.27)) (justify left))
     )
-    (property "Value" "C_Polarized" (at 110.49 61.341 0)
+    (property "Value" "100u" (at 110.49 61.341 0)
       (effects (font (size 1.27 1.27)) (justify left))
     )
@@
       (effects (font (size 1.27 1.27)))
     )
-    (property "Value" "1K8" (at 180.34 76.2 90)
+    (property "Value" "1K" (at 180.34 76.2 90)
       (effects (font (size 1.27 1.27)))
     )
@@
       (effects (font (size 1.27 1.27)) (justify left))
     )
-    (property "Value" "C" (at 99.06 62.23 0)
-      (effects (font (size 1.27 1.27)) (justify left))
-    )
+    (property "Value" "100n" (at 99.06 62.23 0)
+      (effects (font (size 1.27 1.27)) (justify left))
+    )
